File: DMH_VCO_40106_PANEL/DMH_VCO_40106_PANEL.kicad_pcb (KiCad board)
At the start: 2 copper layers, 100 x 200 mm, 35 parts, among them J1 GND

Commit message: Generated VCO Panel Gerbers for test
Other:
- board text removed: "Hard"
- board text removed: "Soft"
