File: DMH_VCO_40106_PANEL/DMH_VCO_40106_PANEL.kicad_sch (KiCad schematic)
At the start: 35 parts, among them J1 GND

Commit message: Updates from testing on breadboard
- Removed Bus CV input, normalled it to V/oct input jack instead
- Renamed Lin FM input to Exp FM In 2
- Added annotations about temporary resistor/pot values
- Added annotations about pots and trimpots pinout
Parts:
- H10, H18: value Exp FM -> Exp FM 1
- H11, H19: value Lin FM -> Exp FM 2
Changed lines of the file:
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@@
 			)
 		)
-		(property "Value" "Lin FM"
+		(property "Value" "Exp FM 2"
 			(at 142.24 58.4199 0)
 			(effects
@@
 			)
 		)
-		(property "Value" "Exp FM"
+		(property "Value" "Exp FM 1"
 			(at 109.22 58.4199 0)
 			(effects
@@
 			)
 		)
-		(property "Value" "Lin FM"
+		(property "Value" "Exp FM 2"
 			(at 139.7 99.0599 0)
 			(effects
@@
 			)
 		)
-		(property "Value" "Exp FM"
+		(property "Value" "Exp FM 1"
 			(at 111.76 99.0599 0)
 			(effects
