File: DMH_VCO_40106_PCB/Inputs_and_Outputs.kicad_sch (KiCad schematic)
At the start: 9 parts, among them J1 Sync, J2 V/Oct, J3 Exp FM, J4 Lin FM, J5 PW Mod, J6 Senoid, J7 Triangle, J8 Square, J9 Sawtooth

Commit message: Updates from testing on breadboard
- Removed Bus CV input, normalled it to V/oct input jack instead
- Renamed Lin FM input to Exp FM In 2
- Added annotations about temporary resistor/pot values
- Added annotations about pots and trimpots pinout
Connections:
- net Bus CV normalled: now reaches J2.TN
- net Exp FM In Jack renamed Exp FM In 1 Jack
- net Lin FM In Jack renamed Exp FM In 2 Jack
- no-connect marks 9 -> 8
Other:
- company: (none) -> DMH Instruments
Changed lines of the file:
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@@
 	(generator_version "8.0")
 	(paper "A4")
+	(title_block
+		(company "DMH Instruments")
+	)
 	(junction
 		(at 165.1 91.44)
@@
 	)
 	(no_connect
-		(at 68.58 77.47)
-	)
-	(no_connect
 		(at 124.46 115.57)
 	)
@@
 	(wire
 		(pts
+			(xy 76.2 80.01) (xy 72.39 80.01)
+		)
+		(stroke
+			(width 0)
+			(type default)
+		)
+	)
+	(wire
+		(pts
 			(xy 165.1 72.39) (xy 165.1 91.44)
 		)
@@
 	(wire
 		(pts
+			(xy 72.39 80.01) (xy 72.39 77.47)
+		)
+		(stroke
+			(width 0)
+			(type default)
+		)
+	)
+	(wire
+		(pts
 			(xy 124.46 113.03) (xy 133.35 113.03)
 		)
@@
 		(pts
 			(xy 101.6 110.49) (xy 101.6 129.54)
+		)
+		(stroke
+			(width 0)
+			(type default)
+		)
+	)
+	(wire
+		(pts
+			(xy 72.39 77.47) (xy 68.58 77.47)
 		)
 		(stroke
@@
 		)
 	)
-	(hierarchical_label "Lin FM In Jack"
+	(hierarchical_label "Exp FM In 2 Jack"
 		(shape output)
 		(at 76.2 113.03 0)
@@
 		)
 	)
+	(hierarchical_label "Bus CV normalled"
+		(shape input)
+		(at 76.2 80.01 0)
+		(fields_autoplaced yes)
+		(effects
+			(font
+				(size 1.27 1.27)
+			)
+			(justify left)
+		)
+	)
 	(hierarchical_label "Sine Out Jack"
 		(shape input)
@@
 		)
 	)
-	(hierarchical_label "Exp FM In Jack"
+	(hierarchical_label "Exp FM In 1 Jack"
 		(shape output)
 		(at 76.2 93.98 0)
