File: DMH_VCO_40106_PCB/Sine_Shaper.kicad_sch (KiCad schematic)
At the start: 13 parts, among them Q5 2N3904, Q6 2N3904, U3 TL072

Commit message: Updates from testing on breadboard
- Removed Bus CV input, normalled it to V/oct input jack instead
- Renamed Lin FM input to Exp FM In 2
- Added annotations about temporary resistor/pot values
- Added annotations about pots and trimpots pinout
Other:
- company: (none) -> DMH Instruments
Changed lines of the file:
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@@
 	(generator_version "8.0")
 	(paper "A4")
+	(title_block
+		(company "DMH Instruments")
+	)
 	(junction
 		(at 176.53 76.2)
