File: DMH_VCO_40106_PCB/Tuner.kicad_sch (KiCad schematic)
At the start: 0 parts

Commit message: Updates from testing on breadboard
- Removed Bus CV input, normalled it to V/oct input jack instead
- Renamed Lin FM input to Exp FM In 2
- Added annotations about temporary resistor/pot values
- Added annotations about pots and trimpots pinout
Other:
- company: (none) -> DMH Instruments
Changed lines of the file:
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@@
 	(generator_version "8.0")
 	(paper "A4")
+	(title_block
+		(company "DMH Instruments")
+	)
 )

Commit message: Added tuner circuit
Parts:
- added C18, C19: 100nF, Capacitor_THT:C_Disc_D4.3mm_W1.9mm_P5.00mm, symbol Device:C
- added D5: 1N4148, Diode_THT:D_DO-35_SOD27_P7.62mm_Horizontal, symbol Diode:1N4148
- added J11: AVR-ISP-6, Connector_IDC:IDC-Header_2x03_P2.54mm_Vertical, symbol Connector:AVR-ISP-6
- added R51, R54, R57: 68k, Resistor_THT:R_Axial_DIN0204_L3.6mm_D1.6mm_P5.08mm_Horizontal, symbol Device:R_US
- added R55, R56: 100k, Resistor_THT:R_Axial_DIN0204_L3.6mm_D1.6mm_P5.08mm_Horizontal, symbol Device:R_US
- added R60, R61, R62, R63, R64, R65, R66, R67: 1k, Resistor_THT:R_Axial_DIN0204_L3.6mm_D1.6mm_P5.08mm_Horizontal, symbol Device:R_US
- added SW3: SW_SPDT, symbol Switch:SW_SPDT_321
- added U5: ATtiny84A-P, Package_DIP:DIP-14_W7.62mm, symbol MCU_Microchip_ATtiny:ATtiny84A-P
- added U6: SM420561N, Display_7Segment:7SegmentLED_LTS6760_LTS6780, symbol Display_Character:SM420561N
Connections:
- new net: R66.1, U5.10 (PA3)
- new net: R66.2, U6.10 (G)
- new net: J11.1 (MISO), R60.1, U5.8 (PA5)
- new net: R60.2, U6.7 (A)
- new net: D5.1 (K), U5.12 (PA1)
- new net: D5.2 (A), R54.2, R56.1, R57.2
- new net: R51.2, R55.1, U5.11 (PA2)
- new net: R64.1, U5.2 (XTAL1/PB0)
- new net: R63.1, U5.3 (XTAL2/PB1)
- new net: J11.5 (~{RST}), U5.4 (~{RESET}/PB3)
- new net: R62.1, U5.5 (PB2)
- new net: R67.1, U5.6 (PA7)
- new net: J11.4 (MOSI), R61.1, U5.7 (PA6)
- new net: J11.3 (SCK), R65.1, U5.9 (PA4)
- new net: R61.2, U6.6 (B)
- new net: R63.2, U6.2 (D)
- new net: R67.2, U6.5 (DP)
- new net: R65.2, U6.9 (F)
- new net: SW3.2 (B), U6.3 (CC), U6.8 (CC)
- new net: R62.2, U6.4 (C)
- new net: R64.2, U6.1 (E)
- new net +5V: C18.1, C19.1, J11.2 (VCC), R55.2, R57.1, U5.1 (VCC)
- new net GND: C18.2, C19.2, J11.6 (GND), R51.1, R56.2, SW3.1 (C), U5.14 (GND)
- new net Sawtooth In: R54.1
Other:
- note added: "Off"
- note added: "On"
